Commit message: 2_mujoco_win_configure

File: urdf/xMateSR4C_gen.urdf (robot description, URDF)
Before this commit: robot xMateSR4C, 8 links, 7 joints
Links:
- link xMateSR4C_base: geometry collision mesh filename=../stl/xMateSR4C_base.stl scale=0.001 0.001 0.001; visual mesh filename=../stl/xMateSR4C_base.stl scale=0.001 0.001 0.001
- link xMateSR4C_link1: geometry collision mesh filename=../stl/xMateSR4C_link1.stl scale=0.001 0.001 0.001; visual mesh filename=../stl/xMateSR4C_link1.stl scale=0.001 0.001 0.001
- link xMateSR4C_link2: geometry collision mesh filename=../stl/xMateSR4C_link2.stl scale=0.001 0.001 0.001; visual mesh filename=../stl/xMateSR4C_link2.stl scale=0.001 0.001 0.001
- link xMateSR4C_link3: geometry collision mesh filename=../stl/xMateSR4C_link3.stl scale=0.001 0.001 0.001; visual mesh filename=../stl/xMateSR4C_link3.stl scale=0.001 0.001 0.001
- link xMateSR4C_link4: geometry collision mesh filename=../stl/xMateSR4C_link4.stl scale=0.001 0.001 0.001; visual mesh filename=../stl/xMateSR4C_link4.stl scale=.001 0.001 0.001
- link xMateSR4C_link5: geometry collision mesh filename=../stl/xMateSR4C_link5.stl scale=0.001 0.001 0.001; visual mesh filename=../stl/xMateSR4C_link5.stl scale=0.001 0.001 0.001
- link xMateSR4C_link6: geometry collision mesh filename=../stl/xMateSR4C_link6.stl scale=0.001 0.001 0.001; visual mesh filename=../stl/xMateSR4C_link6.stl scale=0.001 0.001 0.001

Commit message: 3_change_urdf

File: urdf/xMateSR4C_gen.urdf (robot description, URDF)
Before this commit: robot xMateSR4C, 8 links, 7 joints
Links:
- link xMateSR4C_base: mass 3.44074938 -> 3.16699999486378
Joints:
- joint xmate_joint_2: origin xyz=0 0 0.355 rpy=0 0 0 -> xyz=0 0 0.328 rpy=0 0 0
- joint xmate_joint_3: origin xyz=0.05 0 0.4 rpy=0 0 0 -> xyz=0.050 0 0.4031 rpy=0 0 0
- joint xmate_joint_4: origin xyz=-0.05 0 0.4 rpy=0 0 0 -> xyz=-0.050 0 0.4 rpy=0 0 0
- joint xmate_joint_6: origin xyz=0 0 0.1035 rpy=0.0 0.0 0 -> xyz=0 0 0.1035 rpy=0 0 0
